File: PCB+SCHEMATIC/StratoScience_Template_Board/StratoScience_Template_Board.kicad_pcb (KiCad board)
At the start: 2 copper layers, 63 x 50.5 mm, 7 parts, among them J1 Arduino DC Jack (6-12v)

Commit message: adding stuff
just adding stuff
Parts:
- added G***: LOGO, LOGO, F.Cu at (123.6, 78.8)
- added J2: SD Card, Connector_PinSocket_2.54mm:PinSocket_1x06_P2.54mm_Vertical, F.Cu at (137.9, 79.2)
- added J3: MPU 9250/6500, Connector_PinSocket_2.54mm:PinSocket_1x10_P2.54mm_Vertical, F.Cu at (118.1, 96.8)
- added J4: Tiny_4FSK, Connector_JST:JST_PH_B4B-PH-K_1x04_P2.00mm_Vertical, F.Cu at (168.0, 96.2)
- moved A1 7.51 mm to (147.3, 81.0)
- moved J1 5.09 mm to (133.9, 109.8)
- moved G*** 1.58 mm to (123.5, 88.5)
Connections:
- A1 pad 13: /D10 -> /SD_CS
- A1 pad 14: /D11 -> /SD_MOSI
- A1 pad 15: /D12 -> /SD_MISO
- A1 pad 16: /D13 -> /SD_CLK
- A1 pad 23: /A4 -> /MPU_SDA
- A1 pad 24: /A5 -> /MPU_SCL
Routing:
- net /NANO_VIN: track 0.00 -> 78.5 mm
- net +5V: track 0.00 -> 66.4 mm
- net /MPU_SDA: track 0.00 -> 52.5 mm
- net /SD_CLK: track 0.00 -> 52.4 mm
- net /MPU_SCL: track 0.00 -> 52.3 mm
- net /SD_MISO: track 0.00 -> 41.0 mm
- net +3.3V: track 0.00 -> 40.5 mm
- net /SD_MOSI: track 0.00 -> 32.8 mm
- net /SD_CS: track 0.00 -> 28.2 mm
- net /~{RESET}: track 0.00 -> 15.2 mm
- added copper zone on B.Cu, net Earth
- added copper zone on F.Cu, net Earth
Other:
- board text added: "3 Nerdz press©"
- board text added: "MPU"
- board text added: "NF"
- board text added: "SD"
